File: 0.2/compact/ferris.kicad_pcb (KiCad board)
At the start: 2 copper layers, 208.8 x 86.8 mm, 109 parts, among them J1 TYPE-C-31-M-12, K0_0 KEYSW, K0_1 KEYSW, K0_2 KEYSW, K0_3 KEYSW, K0_4 KEYSW, K0_5 KEYSW, K0_6 KEYSW, K0_7 KEYSW, K0_8 KEYSW, K0_9 KEYSW, K1_0 KEYSW, K1_1 KEYSW, K1_2 KEYSW, K1_3 KEYSW, K1_4 KEYSW, K1_5 KEYSW, K1_6 KEYSW, K1_7 KEYSW, K1_8 KEYSW, K1_9 KEYSW, K2_0 KEYSW, K2_1 KEYSW, K2_2 KEYSW, K2_3 KEYSW, K2_4 KEYSW, K2_5 KEYSW, K2_6 KEYSW, K2_7 KEYSW, K2_8 KEYSW, K2_9 KEYSW, K3_3 KEYSW, K3_4 KEYSW, K3_5 KEYSW, K3_6 KEYSW, Q1 PDTC123JT,215, SW1 B3U-1000P, U1 STM32F072CBT6, U2 MCP23017-E/SO, U3 MCP1700T-3302E/TT, U4 SRV05-4

Commit message: Update to KiCad 7.0
... and prune outdated project files (need to check)
Other:
- net class Default removed
- net class Power removed
